File: DMH_Submodule_VCA/DMH_Submodule_VCA.kicad_pcb (KiCad board)
At the start: 2 copper layers, 41 x 27 mm, 19 parts, among them J1 Conn_02x03_Odd_Even, Q1 BC548, Q2 BC548, U1 TL072

Commit message: Generated VCA gerbers
Other:
- board text added: "Mk1.0 June 2026"
- board text removed: "Mk1.0 - Month Year"
