File: DMH_Submodule_VCA/DMH_Submodule_VCA.kicad_sch (KiCad schematic)
At the start: 34 parts, among them J1 Conn_02x03_Odd_Even, Q1 BC548, Q2 BC548, U1 TL072, U2 TL072

Commit message: Designed PCB
Connections:
- no-connect marks 0 -> 2
