File: DMH_Submodule_VCA/DMH_Submodule_VCA.kicad_sch (KiCad schematic)
At the start: 34 parts, among them J1 Conn_02x03_Odd_Even, Q1 BC548, Q2 BC548, U1 TL072, U2 TL072

Commit message: Swapped J1 and J2 tags around on XFader SM
Other:
- title: (none) -> VCA Submodule
Changed lines of the file:
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@@
 	(paper "A4")
 	(title_block
+		(title "VCA Submodule")
 		(rev "1")
 		(company "DMH Instruments")
-		(comment 1 "PCB for 5 cm Kosmo format synthesizer module")
+		(comment 1 "Submodule PCB Kosmo format synthesizer module")
 	)
 	(circle
