File: DMH_Submodule_XFader/DMH_Submodule_XFader.kicad_pcb (KiCad board)
At the start: 2 copper layers, 41 x 27 mm, 19 parts, among them J1 Conn_02x03_Odd_Even, Q1 BC548, Q2 BC548, U1 TL072

Commit message: Xfader comp placement in progress
Parts:
- removed R1: 100k, Resistor_THT:R_Axial_DIN0207_L6.3mm_D2.5mm_P7.62mm_Horizontal
- added C3: 100nF, Capacitor_THT:C_Disc_D4.3mm_W1.9mm_P5.00mm, F.Cu at (76.2, 83.5)
- added C4: 100nF, Capacitor_THT:C_Disc_D4.3mm_W1.9mm_P5.00mm, F.Cu at (81.2, 97.5)
- added J2: Conn_01x04, Connector_PinHeader_2.54mm:PinHeader_1x04_P2.54mm_Horizontal, F.Cu at (63.1, 63.1)
- added Q3: BC548, Package_TO_SOT_THT:TO-92L_Inline_Wide, F.Cu at (65.0, 72.5)
- added Q4: BC548, Package_TO_SOT_THT:TO-92L_Inline_Wide, F.Cu at (70.0, 72.5)
- added R13: 100R, Resistor_THT:R_Axial_DIN0207_L6.3mm_D2.5mm_P2.54mm_Vertical, F.Cu at (88.8, 85.8)
- added R14: 220k, Resistor_THT:R_Axial_DIN0207_L6.3mm_D2.5mm_P2.54mm_Vertical, F.Cu at (85.8, 61.0)
- added R15: 10k, Resistor_THT:R_Axial_DIN0207_L6.3mm_D2.5mm_P2.54mm_Vertical, F.Cu at (109.2, 51.2)
- added R16: 100k, Resistor_THT:R_Axial_DIN0207_L6.3mm_D2.5mm_P2.54mm_Vertical, F.Cu at (122.5, 65.3)
- added R18: 100k, Resistor_THT:R_Axial_DIN0207_L6.3mm_D2.5mm_P2.54mm_Vertical, F.Cu at (122.5, 69.3)
- added R19: 82k, Resistor_THT:R_Axial_DIN0207_L6.3mm_D2.5mm_P2.54mm_Vertical, F.Cu at (122.5, 73.4)
- added R20: 100k, Resistor_THT:R_Axial_DIN0207_L6.3mm_D2.5mm_P2.54mm_Vertical, F.Cu at (122.5, 77.4)
- added R21: 100k, Resistor_THT:R_Axial_DIN0207_L6.3mm_D2.5mm_P2.54mm_Vertical, F.Cu at (133.2, 53.1)
- added R22: 20k, Resistor_THT:R_Axial_DIN0207_L6.3mm_D2.5mm_P2.54mm_Vertical, F.Cu at (133.2, 57.2)
- added R23: 20k, Resistor_THT:R_Axial_DIN0207_L6.3mm_D2.5mm_P2.54mm_Vertical, F.Cu at (133.2, 61.2)
- added R24: 100k, Resistor_THT:R_Axial_DIN0207_L6.3mm_D2.5mm_P2.54mm_Vertical, F.Cu at (133.2, 65.3)
- added R25: 10k, Resistor_THT:R_Axial_DIN0207_L6.3mm_D2.5mm_P2.54mm_Vertical, F.Cu at (133.2, 69.3)
- added R26: 10k, Resistor_THT:R_Axial_DIN0207_L6.3mm_D2.5mm_P2.54mm_Vertical, F.Cu at (133.2, 73.4)
- added R27: 100k, Resistor_THT:R_Axial_DIN0207_L6.3mm_D2.5mm_P2.54mm_Vertical, F.Cu at (133.2, 77.4)
- added R28: 100k, Resistor_THT:R_Axial_DIN0207_L6.3mm_D2.5mm_P2.54mm_Vertical, F.Cu at (144.0, 53.1)
- added R29: 100k, Resistor_THT:R_Axial_DIN0207_L6.3mm_D2.5mm_P2.54mm_Vertical, F.Cu at (108.5, 58.5)
- added R30: 100R, Resistor_THT:R_Axial_DIN0207_L6.3mm_D2.5mm_P2.54mm_Vertical, F.Cu at (144.0, 61.2)
- added R31: 100R, Resistor_THT:R_Axial_DIN0207_L6.3mm_D2.5mm_P2.54mm_Vertical, F.Cu at (144.0, 65.3)
- added R32: 110k, Resistor_THT:R_Axial_DIN0207_L6.3mm_D2.5mm_P2.54mm_Vertical, F.Cu at (144.0, 69.3)
- added R33: 10k, Resistor_THT:R_Axial_DIN0207_L6.3mm_D2.5mm_P2.54mm_Vertical, F.Cu at (144.0, 73.4)
- added R34: 100k, Resistor_THT:R_Axial_DIN0207_L6.3mm_D2.5mm_P2.54mm_Vertical, F.Cu at (144.0, 77.4)
- added RV2: 100k, Potentiometer_THT:Potentiometer_Bourns_3296X_Horizontal, F.Cu at (89.8, 60.7)
- added RV3: 50k, Potentiometer_THT:Potentiometer_Bourns_3296X_Horizontal, F.Cu at (89.8, 90.5)
- added U2: TL072, Package_DIP:DIP-8_W7.62mm_Socket, F.Cu at (74.9, 86.7)
- J1: value Conn_02x03_Odd_Even -> Conn_01x08; footprint Connector_PinHeader_2.54mm:PinHeader_2x03_P2.54mm_Horizontal -> Connector_PinHeader_2.54mm:PinHeader_1x08_P2.54mm_Horizontal
- R10, R11, R8: footprint Resistor_THT:R_Axial_DIN0207_L6.3mm_D2.5mm_P7.62mm_Horizontal -> Resistor_THT:R_Axial_DIN0207_L6.3mm_D2.5mm_P2.54mm_Vertical
- R12: value 100k -> 100R; footprint Resistor_THT:R_Axial_DIN0207_L6.3mm_D2.5mm_P7.62mm_Horizontal -> Resistor_THT:R_Axial_DIN0207_L6.3mm_D2.5mm_P2.54mm_Vertical
- R2: value 100k -> 20k; footprint Resistor_THT:R_Axial_DIN0207_L6.3mm_D2.5mm_P7.62mm_Horizontal -> Resistor_THT:R_Axial_DIN0207_L6.3mm_D2.5mm_P2.54mm_Vertical
- R3: value 100R -> 20k; footprint Resistor_THT:R_Axial_DIN0207_L6.3mm_D2.5mm_P7.62mm_Horizontal -> Resistor_THT:R_Axial_DIN0207_L6.3mm_D2.5mm_P2.54mm_Vertical
- R4: value 20k -> 33k; footprint Resistor_THT:R_Axial_DIN0207_L6.3mm_D2.5mm_P7.62mm_Horizontal -> Resistor_THT:R_Axial_DIN0207_L6.3mm_D2.5mm_P2.54mm_Vertical
- R5, R9: value 10k -> 100k; footprint Resistor_THT:R_Axial_DIN0207_L6.3mm_D2.5mm_P7.62mm_Horizontal -> Resistor_THT:R_Axial_DIN0207_L6.3mm_D2.5mm_P2.54mm_Vertical
- R6: value 20k -> 100k; footprint Resistor_THT:R_Axial_DIN0207_L6.3mm_D2.5mm_P7.62mm_Horizontal -> Resistor_THT:R_Axial_DIN0207_L6.3mm_D2.5mm_P2.54mm_Vertical
- R7: value 100R -> 10k; footprint Resistor_THT:R_Axial_DIN0207_L6.3mm_D2.5mm_P7.62mm_Horizontal -> Resistor_THT:R_Axial_DIN0207_L6.3mm_D2.5mm_P2.54mm_Vertical
- U1: value TL072 -> TL074; footprint Package_DIP:DIP-8_W7.62mm_Socket -> Package_DIP:DIP-14_W7.62mm_Socket
- moved R4 94.4 mm to (139.3, 109.3), turned to 0 degrees
- moved R9 93.1 mm to (139.3, 129.6), turned to 0 degrees
- moved R6 92.3 mm to (139.3, 117.4), turned to 0 degrees
- moved R5 87.7 mm to (139.3, 113.4), turned to 0 degrees
- moved R8 87.5 mm to (139.3, 125.5), turned to 0 degrees
- moved R3 85.4 mm to (139.3, 105.3), turned to 0 degrees
- moved R7 81.4 mm to (139.3, 121.5), turned to 0 degrees
- moved R2 70.1 mm to (139.3, 101.2), turned to 0 degrees
- moved R10 40.3 mm to (93.8, 84.0), turned to -90 degrees
- moved J1 38.7 mm to (63.1, 94.4), turned to 180 degrees
- moved RV1 26.9 mm to (89.8, 55.3), turned to 180 degrees
- moved Q1 26.4 mm to (95.0, 74.5)
- moved Q2 19.6 mm to (90.0, 74.5)
- moved R11 18.6 mm to (88.7, 65.2), turned to 0 degrees
- moved R12 16.2 mm to (100.7, 65.0), turned to 0 degrees
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Connections:
- J1 pad 1: +12V -> /In A
- J1 pad 2: /CV Mix In -> /Out A
- J1 pad 3: -12V -> /In B
- J1 pad 4: /Signal In -> /Out B
- J1 pad 5: GND -> /CV Att In
- J1 pad 6: /Signal Out -> /CV Att Pot
- R10 pad 1: Net-(R10-Pad1) -> Net-(Q1-B)
- R10 pad 2: Net-(Q2-B) -> /In A
- R11 pad 1: Net-(U1B-+) -> Net-(R11-Pad1)
- R11 pad 2: GND -> Net-(Q2-B)
- R12 pad 1: /Signal Out -> GND
- R12 pad 2: Net-(U1B--) -> Net-(Q1-B)
- R2 pad 1: Net-(Q1-B) -> Net-(Q1-C)
- R2 pad 2: /Signal In -> +12V
- R3 pad 1: GND -> Net-(Q2-C)
- R3 pad 2: Net-(Q1-B) -> +12V
- R4 pad 1: Net-(Q1-C) -> /CV Att In
- R4 pad 2: +12V -> Net-(U2B--)
- R5 pad 1: Net-(R1-Pad2) -> /CV Mix In
- R5 pad 2: Net-(Q1-E) -> Net-(R5-Pad2)
- R6 pad 1: Net-(Q2-C) -> /Out A
- R6 pad 2: +12V -> Net-(U1C--)
- R7 pad 1: GND -> Net-(U1C--)
- R7 pad 2: Net-(Q2-B) -> Net-(Q2-C)
- R8 pad 1: Net-(U1B--) -> Net-(U1C-+)
- R9 pad 1: Net-(U1B-+) -> Net-(U1C-+)
- R9 pad 2: Net-(Q2-C) -> GND
- RV1 pad 2: Net-(R10-Pad1) -> Net-(R11-Pad1)
- U1 pad 1: Net-(R1-Pad2) -> Net-(R33-Pad1)
- U1 pad 2: /CV Mix In -> Net-(U1A--)
- U1 pad 4: -12V -> +12V
- U1 pad 7: /Signal Out -> /Out B
- U1 pad 8: +12V -> /Out A
Routing:
- net +12V: track 49.7 -> 0.00 mm
- net -12V: track 48.4 -> 0.00 mm
- net Net-(Q2-B): track 38.2 -> 0.00 mm
- net Net-(R1-Pad2): track 31.9 -> 0.00 mm
- net /CV Mix In: track 29.1 -> 0.00 mm
- net Net-(U1B-+): track 27.2 -> 0.00 mm
- net Net-(Q1-B): track 25.8 -> 0.00 mm
- net Net-(Q2-C): track 20.2 -> 0.00 mm
- net Net-(Q1-C): track 17.1 -> 0.00 mm
- net Net-(U1B--): track 16.3 -> 0.00 mm
- net /Signal Out: track 13.7 -> 0.00 mm
- net Net-(R10-Pad1): track 12.1 -> 0.00 mm
- net Net-(Q1-E): track 11.5 -> 0.00 mm
- net /Signal In: track 8.65 -> 0.00 mm
Other:
- board size 41 x 27 mm -> 37.5 x 62.5 mm

Commit message: Xfader comp placement in progress
Parts:
- moved R20 53.3 mm to (71.8, 61.0), turned to 90 degrees
- moved R15 34.2 mm to (85.8, 76.2), turned to -90 degrees
- moved R29 22.7 mm to (87.0, 65.5)
- moved R13 16.5 mm to (93.5, 70.0), turned to 0 degrees
- moved R12 14.6 mm to (87.0, 70.0)
- moved R10 14.0 mm to (90.3, 97.5), turned to 180 degrees
- moved Q2 7.43 mm to (95.2, 79.8)
- moved Q1 7.09 mm to (90.2, 79.8)
- moved R11 4.76 mm to (93.5, 65.5)
Connections:
- R29 pad 1: Net-(R29-Pad1) -> Net-(Q4-B)
- R29 pad 2: Net-(Q4-B) -> Net-(R29-Pad2)
- RV2 pad 2: Net-(R29-Pad1) -> Net-(R29-Pad2)
Changed lines of the file:
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@@
 	(footprint "Resistor_THT:R_Axial_DIN0207_L6.3mm_D2.5mm_P2.54mm_Vertical"
 		(layer "F.Cu")
-		(at 88.75 85.795 90)
+		(at 93.455 70)
 		(descr "Resistor, Axial_DIN0207 series, Axial, Vertical, pin pitch=2.54mm, 0.25W = 1/4W, length*diameter=6.3*2.5mm^2, http://cdn-reichelt.de/documents/datenblatt/B400/1_4W%23YAG.pdf")
 		(tags "Resistor Axial_DIN0207 series Axial Vertical pin pitch 2.54mm 0.25W = 1/4W length 6.3mm diameter 2.5mm")
 		(property "Reference" "R13"
-			(at 4.295 0 0)
+			(at -2.205 0 90)
 			(layer "F.SilkS")
 			(effects
@@
 		)
 		(property "Value" "100R"
-			(at 1.295 2.25 90)
+			(at 1.295 2.25 0)
 			(layer "F.SilkS")
 			(effects
@@
 		)
 		(property "Datasheet" ""
-			(at 0 0 90)
+			(at 0 0 0)
 			(layer "F.Fab")
 			(hide yes)
@@
 		)
 		(property "Description" "Resistor, US symbol"
-			(at 0 0 90)
+			(at 0 0 0)
 			(layer "F.Fab")
 			(hide yes)
@@
 		)
 		(property "KiLib_Generator" "resistor/THT"
-			(at 0 0 90)
+			(at 0 0 0)
 			(layer "F.SilkS")
 			(hide yes)
@@
 		)
 		(fp_text user "${REFERENCE}"
-			(at 1.27 -2.37 90)
+			(at 1.27 -2.37 0)
 			(layer "F.Fab")
 			(effects
@@
 		)
 		(pad "1" thru_hole circle
-			(at 0 0 90)
+			(at 0 0)
 			(size 1.6 1.6)
 			(drill 0.8)
@@
 		)
 		(pad "2" thru_hole circle
-			(at 2.54 0 90)
+			(at 2.54 0)
 			(size 1.6 1.6)
 			(drill 0.8)
@@
 	(footprint "Resistor_THT:R_Axial_DIN0207_L6.3mm_D2.5mm_P2.54mm_Vertical"
 		(layer "F.Cu")
-		(at 93.75 83.955 -90)
+		(at 90.295 97.5 180)
 		(descr "Resistor, Axial_DIN0207 series, Axial, Vertical, pin pitch=2.54mm, 0.25W = 1/4W, length*diameter=6.3*2.5mm^2, http://cdn-reichelt.de/documents/datenblatt/B400/1_4W%23YAG.pdf")
 		(tags "Resistor Axial_DIN0207 series Axial Vertical pin pitch 2.54mm 0.25W = 1/4W length 6.3mm diameter 2.5mm")
 		(property "Reference" "R10"
-			(at -2.205 0 180)
+			(at 4.295 0 90)
 			(layer "F.SilkS")
 			(effects
@@
 		)
 		(property "Value" "100k"
-			(at 1.295 -2.25 270)
+			(at 1.295 -2.25 0)
 			(layer "F.SilkS")
 			(effects
@@
 		)
 		(property "Datasheet" ""
-			(at 0 0 90)
+			(at 0 0 0)
 			(layer "F.Fab")
 			(hide yes)
@@
 		)
 		(property "Description" "Resistor, US symbol"
-			(at 0 0 90)
+			(at 0 0 0)
 			(layer "F.Fab")
 			(hide yes)
@@
 		)
 		(property "KiLib_Generator" "resistor/THT"
-			(at 0 0 90)
+			(at 0 0 0)
 			(layer "F.SilkS")
 			(hide yes)
@@
 		)
 		(property "Function" ""
-			(at 0 0 270)
+			(at 0 0 180)
 			(unlocked yes)
 			(layer "F.Fab")
@@
 		)
 		(fp_text user "${REFERENCE}"
-			(at 1.27 -2.37 90)
+			(at 1.27 -2.37 0)
 			(layer "F.Fab")
 			(effects
@@
 		)
 		(pad "1" thru_hole circle
-			(at 0 0 270)
+			(at 0 0 180)
 			(size 1.6 1.6)
 			(drill 0.8)
@@
 		)
 		(pad "2" thru_hole circle
-			(at 2.54 0 270)
+			(at 2.54 0 180)
 			(size 1.6 1.6)
 			(drill 0.8)
@@
 			(layers "*.Cu" "*.Mask")
 			(remove_unused_layers no)
-			(net "Net-(R29-Pad1)")
+			(net "Net-(R29-Pad2)")
 			(pinfunction "2_2")
 			(pintype "passive")
@@
 	(footprint "Resistor_THT:R_Axial_DIN0207_L6.3mm_D2.5mm_P2.54mm_Vertical"
 		(layer "F.Cu")
-		(at 108.5 58.5)
+		(at 86.955 65.5)
 		(descr "Resistor, Axial_DIN0207 series, Axial, Vertical, pin pitch=2.54mm, 0.25W = 1/4W, length*diameter=6.3*2.5mm^2, http://cdn-reichelt.de/documents/datenblatt/B400/1_4W%23YAG.pdf")
 		(tags "Resistor Axial_DIN0207 series Axial Vertical pin pitch 2.54mm 0.25W = 1/4W length 6.3mm diameter 2.5mm")
 		(property "Reference" "R29"
-			(at 1.27 -2.37 0)
+			(at -2.205 0 90)
 			(layer "F.SilkS")
 			(effects
@@
 		)
 		(property "Value" "100k"
-			(at 1.27 2.37 0)
+			(at 1.295 2.25 0)
 			(layer "F.SilkS")
 			(effects
@@
 			(layers "*.Cu" "*.Mask")
 			(remove_unused_layers no)
-			(net "Net-(R29-Pad1)")
+			(net "Net-(Q4-B)")
 			(pintype "passive")
 		)
@@
 			(layers "*.Cu" "*.Mask")
 			(remove_unused_layers no)
-			(net "Net-(Q4-B)")
+			(net "Net-(R29-Pad2)")
 			(pintype "passive")
 		)
@@
 	(footprint "Package_TO_SOT_THT:TO-92L_Inline_Wide"
 		(layer "F.Cu")
-		(at 94.95 74.54 90)
+		(at 90.2 79.8 90)
 		(descr "TO-92L leads in-line (large body variant of TO-92), also known as TO-226, wide, drill 0.75mm (see https://www.diodes.com/assets/Package-Files/TO92L.pdf and http://www.ti.com/lit/an/snoa059/snoa059.pdf)")
 		(tags "TO-92L Inline Wide transistor")
 		(property "Reference" "Q1"
-			(at 5.55 -2.355 90)
+			(at 5.8 -1.95 90)
 			(layer "F.SilkS")
 			(effects
@@
 	(footprint "Package_TO_SOT_THT:TO-92L_Inline_Wide"
 		(layer "F.Cu")
-		(at 89.95 74.54 90)
+		(at 95.2 79.8 90)
 		(descr "TO-92L leads in-line (large body variant of TO-92), also known as TO-226, wide, drill 0.75mm (see https://www.diodes.com/assets/Package-Files/TO92L.pdf and http://www.ti.com/lit/an/snoa059/snoa059.pdf)")
 		(tags "TO-92L Inline Wide transistor")
 		(property "Reference" "Q2"
-			(at 5.55 -2.355 90)
+			(at 5.8 -1.95 90)
 			(layer "F.SilkS")
 			(effects
@@
 	(footprint "Resistor_THT:R_Axial_DIN0207_L6.3mm_D2.5mm_P2.54mm_Vertical"
 		(layer "F.Cu")
-		(at 109.205 51.25)
+		(at 85.75 76.205 -90)
 		(descr "Resistor, Axial_DIN0207 series, Axial, Vertical, pin pitch=2.54mm, 0.25W = 1/4W, length*diameter=6.3*2.5mm^2, http://cdn-reichelt.de/documents/datenblatt/B400/1_4W%23YAG.pdf")
 		(tags "Resistor Axial_DIN0207 series Axial Vertical pin pitch 2.54mm 0.25W = 1/4W length 6.3mm diameter 2.5mm")
 		(property "Reference" "R15"
-			(at 1.27 -2.37 0)
+			(at 4.295 0 180)
 			(layer "F.SilkS")
 			(effects
@@
 		)
 		(property "Value" "10k"
-			(at 1.27 2.37 0)
+			(at 1.27 2.37 90)
 			(layer "F.SilkS")
 			(effects
@@
 		)
 		(property "Datasheet" ""
-			(at 0 0 0)
+			(at 0 0 90)
 			(layer "F.Fab")
 			(hide yes)
@@
 		)
 		(property "Description" "Resistor, US symbol"
-			(at 0 0 0)
+			(at 0 0 90)
 			(layer "F.Fab")
 			(hide yes)
@@
 		)
 		(property "KiLib_Generator" "resistor/THT"
-			(at 0 0 0)
+			(at 0 0 90)
 			(layer "F.SilkS")
 			(hide yes)
@@
 		)
 		(fp_text user "${REFERENCE}"
-			(at 1.27 -2.37 0)
+			(at 1.27 -2.37 90)
 			(layer "F.Fab")
 			(effects
@@
 		)
 		(pad "1" thru_hole circle
-			(at 0 0)
+			(at 0 0 270)
 			(size 1.6 1.6)
 			(drill 0.8)
@@
 		)
 		(pad "2" thru_hole circle
-			(at 2.54 0)
+			(at 2.54 0 270)
 			(size 1.6 1.6)
 			(drill 0.8)
@@
 		(tags "THT DIP DIL PDIP 2.54mm 7.62mm 300mil Socket")
 		(property "Reference" "U1"
-			(at -0.69 -2.585 0)
+			(at -0.44 -2.585 90)
 			(layer "F.SilkS")
 			(effects
@@
 	(footprint "Resistor_THT:R_Axial_DIN0207_L6.3mm_D2.5mm_P2.54mm_Vertical"
 		(layer "F.Cu")
-		(at 88.705 65.25)
+		(at 93.455 65.5)
 		(descr "Resistor, Axial_DIN0207 series, Axial, Vertical, pin pitch=2.54mm, 0.25W = 1/4W, length*diameter=6.3*2.5mm^2, http://cdn-reichelt.de/documents/datenblatt/B400/1_4W%23YAG.pdf")
 		(tags "Resistor Axial_DIN0207 series Axial Vertical pin pitch 2.54mm 0.25W = 1/4W length 6.3mm diameter 2.5mm")
@@
 		)
 		(property "Value" "100k"
-			(at 1.295 -2.25 0)
+			(at 1.295 2.25 0)
 			(layer "F.SilkS")
 			(effects
@@
 	(footprint "Resistor_THT:R_Axial_DIN0207_L6.3mm_D2.5mm_P2.54mm_Vertical"
 		(layer "F.Cu")
-		(at 100.705 65)
+		(at 86.955 70)
 		(descr "Resistor, Axial_DIN0207 series, Axial, Vertical, pin pitch=2.54mm, 0.25W = 1/4W, length*diameter=6.3*2.5mm^2, http://cdn-reichelt.de/documents/datenblatt/B400/1_4W%23YAG.pdf")
 		(tags "Resistor Axial_DIN0207 series Axial Vertical pin pitch 2.54mm 0.25W = 1/4W length 6.3mm diameter 2.5mm")
 		(property "Reference" "R12"
-			(at 4.295 0 90)
+			(at -2.205 0 90)
 			(layer "F.SilkS")
 			(effects
@@
 	(footprint "Resistor_THT:R_Axial_DIN0207_L6.3mm_D2.5mm_P2.54mm_Vertical"
 		(layer "F.Cu")
-		(at 122.475 77.425)
+		(at 71.75 61.04 90)
 		(descr "Resistor, Axial_DIN0207 series, Axial, Vertical, pin pitch=2.54mm, 0.25W = 1/4W, length*diameter=6.3*2.5mm^2, http://cdn-reichelt.de/documents/datenblatt/B400/1_4W%23YAG.pdf")
 		(tags "Resistor Axial_DIN0207 series Axial Vertical pin pitch 2.54mm 0.25W = 1/4W length 6.3mm diameter 2.5mm")
 		(property "Reference" "R20"
-			(at 1.27 -2.37 0)
+			(at -2.205 0 180)
 			(layer "F.SilkS")
 			(effects
@@
 		)
 		(property "Value" "100k"
-			(at 1.27 2.37 0)
+			(at 4.295 0 180)
 			(layer "F.SilkS")
 			(effects
@@
 		)
 		(property "Datasheet" ""
-			(at 0 0 0)
+			(at 0 0 90)
 			(layer "F.Fab")
 			(hide yes)
@@
 		)
 		(property "Description" "Resistor, US symbol"
-			(at 0 0 0)
+			(at 0 0 90)
 			(layer "F.Fab")
 			(hide yes)
@@
 		)
 		(property "KiLib_Generator" "resistor/THT"
-			(at 0 0 0)
+			(at 0 0 90)
 			(layer "F.SilkS")
 			(hide yes)
@@
 		)
 		(fp_text user "${REFERENCE}"
-			(at 1.27 -2.37 0)
+			(at 1.27 -2.37 90)
 			(layer "F.Fab")
 			(effects
@@
 		)
 		(pad "1" thru_hole circle
-			(at 0 0)
+			(at 0 0 90)
 			(size 1.6 1.6)
 			(drill 0.8)
@@
 		)
 		(pad "2" thru_hole circle
-			(at 2.54 0)
+			(at 2.54 0 90)
 			(size 1.6 1.6)
 			(drill 0.8)
