File: DMH_Submodule_XFader/DMH_Submodule_XFader.kicad_sch (KiCad schematic)
At the start: 46 parts, among them J1 Conn_02x03_Odd_Even, Q1 BC548, Q2 BC548, Q3 BC548, Q4 BC548, U1 TL072, U2 TL072, U3 TL072

Commit message: Designed X fader schematic
Parts:
- removed J1: Conn_02x03_Odd_Even, Connector_PinHeader_2.54mm:PinHeader_2x03_P2.54mm_Horizontal, symbol Connector_Generic:Conn_02x03_Odd_Even
- removed RV3: 100k, SynthStuff:Potentiometer_TT_P110KH1, symbol Device:R_Potentiometer_US
- removed RV5: 50k, Potentiometer_THT:Potentiometer_Bourns_3296W_Vertical, symbol Device:R_Potentiometer_Trim_US
- removed U1, U2: TL072, Package_DIP:DIP-8_W7.62mm_Socket, symbol Amplifier_Operational:TL072
- added J1: Conn_01x08, Connector_PinHeader_2.54mm:PinHeader_1x08_P2.54mm_Vertical, symbol Connector_Generic:Conn_01x08
- added J2: Conn_01x04, Connector_PinHeader_2.54mm:PinHeader_1x04_P2.54mm_Vertical, symbol Connector_Generic:Conn_01x04
- added R14, R17: 220k, Resistor_THT:R_Axial_DIN0207_L6.3mm_D2.5mm_P7.62mm_Horizontal, symbol Device:R_US
- added R19: 82k, Resistor_THT:R_Axial_DIN0207_L6.3mm_D2.5mm_P7.62mm_Horizontal, symbol Device:R_US
- added R21, R5: 100k, Resistor_THT:R_Axial_DIN0207_L6.3mm_D2.5mm_P7.62mm_Horizontal, symbol Device:R_US
- added R32: 110k, Resistor_THT:R_Axial_DIN0207_L6.3mm_D2.5mm_P7.62mm_Horizontal, symbol Device:R_US
- added RV5: 100k, SynthStuff:Potentiometer_TT_P110KH1, symbol Device:R_Potentiometer_US
- added U1: TL074, Package_DIP:DIP-14_W7.62mm_Socket, symbol Amplifier_Operational:TL074
- R18: renamed from R26; value 33k -> 100k
- RV1: Function Symmetry -> Symmetry A
- RV2: Function Symmetry -> Symmetry B
- RV3: renamed from RV6; Function Zero adj B -> Zero adj
- RV4: Function CV Amt B -> CV Amt
- renumbered C3 to C2, C2 to C3, R19 to R1, R2 to R10, R10 to R11, R3 to R12, R7 to R13, R5 to R15, R1 to R16, R4 to R2, R28 to R20, R16 to R22, R18 to R23, R25 to R24, R21 to R25, R22 to R26, R24 to R27, R14 to R28, R23 to R29, R6 to R3, R15 to R30, R20 to R31, R17 to R33, R13 to R34, R27 to R4, R12 to R6, R8 to R7, R9 to R8, R11 to R9, U3 to U2
Connections:
- net Signal Out A is gone; now on net Out A: R6.1
- net +12V: now also C3.1, J2.1 (Pin_1), R14.2, R32.2, RV5.3, U1.4 (V+); no longer C2.1
- net -12V: now also C2.2, J2.2 (Pin_2), RV5.1, U1.11 (V-); no longer C3.2
- net CV Mix In: now also J1.7 (Pin_7), R14.1, R17.2, R5.1, U1.13 (-)
- net GND: now also C2.1, C3.2, U2.3 (+), J2.3 (Pin_3), J2.4 (Pin_4), U1.12 (+), U1.3 (+); no longer C2.2, C3.1
- net at R6.2, R7.1: now also U1.9 (-)
- net at R20.1, R34.1: now also R32.1, U1.2 (-)
- net at R33.1, R34.2: now also U1.1
- net at Q3.1 (C), R22.1: now also R26.2; no longer R25.2
- net at R15.1, R16.2, R20.2: now also U1.14
- net at R18.2, U2.2 (-): now also R19.1, R21.2
- net at Q4.1 (C), R23.1: now also R25.2; no longer R26.2
- net CV Att Pot: now reaches RV4.2, U2.5 (+)
- net CV Att Pot: now also J1.6 (Pin_6)
- net at R26.1, R27.1: now also U1.5 (+)
- net at R24.2, R25.1: now also U1.6 (-)
- net at R8.1, R9.1: now also U1.10 (+)
- net at Q2.1 (C), R3.1: now also R7.2; no longer R8.2
- net at Q1.1 (C), R2.1: now also R8.2; no longer R7.2
- net CV_Att_A renamed Out X
- net Out X: now also J1.8 (Pin_8), R19.2
- net CV_Att_B: no longer names the net of RV3.2, RV3.3, U2.7
- net CV_Att_B: now also R5.2
- net CV_In_A renamed Out A
- net Out A: now also J1.2 (Pin_2), R21.1, U1.8
- net CV_In_B renamed CV Att In
- net CV Att In: now also J1.5 (Pin_5)
- net Signal In A renamed In A
- net In A: now also J1.1 (Pin_1)
- net Signal In B renamed In B
- net In B: now also J1.3 (Pin_3)
- net Signal Out B renamed Out B
- net Out B: now also J1.4 (Pin_4), U1.7
- new net: R17.1, RV5.2
Other:
- note added: "If no Attenuverter pot is used, pin "CV Att Pot" shall be connected directly to GND."
- note added: "Pot at center = both VCAs half open (when other CV sources are 0V or disconnected)"
- moved on the sheet: C1, C2, C3, C4, R1, R16, R18, R20, R34, R4, RV3, RV4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

Commit message: Xfader comp placement in progress
Parts:
- J1: footprint Connector_PinHeader_2.54mm:PinHeader_1x08_P2.54mm_Vertical -> Connector_PinHeader_2.54mm:PinHeader_1x08_P2.54mm_Horizontal
- J2: footprint Connector_PinHeader_2.54mm:PinHeader_1x04_P2.54mm_Vertical -> Connector_PinHeader_2.54mm:PinHeader_1x04_P2.54mm_Horizontal
- R10, R11, R12, R13, R14, R15, R16, R18, R19, R2, R20, R21, R22, R23, R24, R25, R26, R27, R28, R29, R3, R30, R31, R32, R33, R34, R4, R5, R6, R7, R8, R9: footprint Resistor_THT:R_Axial_DIN0207_L6.3mm_D2.5mm_P7.62mm_Horizontal -> Resistor_THT:R_Axial_DIN0207_L6.3mm_D2.5mm_P2.54mm_Vertical
- RV3: footprint Potentiometer_THT:Potentiometer_Bourns_3296W_Vertical -> Potentiometer_THT:Potentiometer_Bourns_3296X_Horizontal
Connections:
- net +12V: now also J2.2 (Pin_2); no longer J2.1 (Pin_1)
- net -12V: now also J2.3 (Pin_3); no longer J2.2 (Pin_2)
- net GND: now also J2.1 (Pin_1); no longer J2.3 (Pin_3)

Commit message: Xfader comp placement in progress
Connections:
- net at Q4.2 (B), R31.2: now also R29.1; no longer R29.2
- net at RV2.2: now also R29.2; no longer R29.1
Other:
- moved on the sheet: R29
Changed lines of the file:
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@@
 	(symbol
 		(lib_id "Device:R_US")
-		(at 196.85 228.6 270)
+		(at 196.85 228.6 90)
+		(mirror x)
 		(unit 1)
 		(body_style 1)
@@
 		(in_pos_files yes)
 		(dnp no)
-		(fields_autoplaced yes)
 		(property "Reference" "R29"
 			(at 196.85 222.25 90)
@@
 		)
 		(property "Footprint" "Resistor_THT:R_Axial_DIN0207_L6.3mm_D2.5mm_P2.54mm_Vertical"
-			(at 196.596 229.616 90)
+			(at 197.104 229.616 90)
 			(hide yes)
 			(show_name no)
