File: DMH_Submodule_XFader/DMH_Submodule_XFader.kicad_sch (KiCad schematic)
At the start: 51 parts, among them J1 Conn_01x08, J2 Conn_01x04, Q1 BC548, Q2 BC548, Q3 BC548, Q4 BC548, U1 TL074, U2 TL072

Commit message: Xfader comp placement done
Connections:
- net +12V: now also R2.1, R22.1, R23.1, R3.1; no longer R2.2, R22.2, R23.2, R3.2
- net CV Att In: now also R4.2; no longer R4.1
- net Out A: now also R18.2, R21.2; no longer R18.1, R21.1
- net at Q3.1 (C), R26.2: now also R22.2; no longer R22.1
- net at Q4.1 (C), R25.2: now also R23.2; no longer R23.1
- net at RV3.1, U2.6 (-): now also R4.1; no longer R4.2
- net at R19.1, U2.2 (-): now also R18.1, R21.1; no longer R18.2, R21.2
- net at Q1.1 (C), R8.2: now also R2.2; no longer R2.1
- net at Q2.1 (C), R7.2: now also R3.2; no longer R3.1
Other:
- moved on the sheet: R18, R2, R21, R22, R4
Changed lines of the file:
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@@
 	)
 	(junction
+		(at 66.04 204.47)
+		(diameter 0)
+		(color 0 0 0 0)
+	)
+	(junction
 		(at 101.6 114.3)
 		(diameter 0)
@@
 	)
 	(junction
-		(at 63.5 204.47)
-		(diameter 0)
-		(color 0 0 0 0)
-	)
-	(junction
 		(at 25.4 252.73)
 		(diameter 0)
@@
 	(wire
 		(pts
-			(xy 63.5 204.47) (xy 63.5 208.28)
-		)
-		(stroke
-			(width 0)
-			(type default)
-		)
-	)
-	(wire
-		(pts
 			(xy 96.52 124.46) (xy 101.6 124.46)
 		)
@@
 	(wire
 		(pts
+			(xy 45.72 207.01) (xy 50.8 207.01)
+		)
+		(stroke
+			(width 0)
+			(type default)
+		)
+	)
+	(wire
+		(pts
 			(xy 77.47 25.4) (xy 77.47 35.56)
 		)
@@
 	(wire
 		(pts
-			(xy 43.18 204.47) (xy 63.5 204.47)
+			(xy 43.18 204.47) (xy 66.04 204.47)
 		)
 		(stroke
@@
 	(wire
 		(pts
+			(xy 66.04 204.47) (xy 66.04 208.28)
+		)
+		(stroke
+			(width 0)
+			(type default)
+		)
+	)
+	(wire
+		(pts
 			(xy 121.92 127) (xy 127 127)
 		)
@@
 		(in_pos_files yes)
 		(dnp no)
-		(fields_autoplaced yes)
 		(property "Reference" "R10"
 			(at 133.35 82.55 90)
@@
 		(lib_id "Device:R_US")
 		(at 177.8 171.45 0)
-		(mirror x)
 		(unit 1)
 		(body_style 1)
@@
 		(dnp no)
 		(property "Reference" "R23"
-			(at 175.26 170.1799 0)
+			(at 175.26 172.7201 0)
 			(show_name no)
 			(do_not_autoplace no)
@@
 		)
 		(property "Value" "20k"
-			(at 175.26 172.7199 0)
+			(at 175.26 170.1801 0)
 			(show_name no)
 			(do_not_autoplace no)
@@
 		)
 		(property "Footprint" "Resistor_THT:R_Axial_DIN0207_L6.3mm_D2.5mm_P2.54mm_Vertical"
-			(at 178.816 171.196 90)
+			(at 178.816 171.704 90)
 			(hide yes)
 			(show_name no)
@@
 	(symbol
 		(lib_id "power:PWR_FLAG")
-		(at 63.5 204.47 270)
+		(at 66.04 204.47 270)
 		(unit 1)
 		(body_style 1)
@@
 		(fields_autoplaced yes)
 		(property "Reference" "#FLG02"
-			(at 65.405 204.47 0)
+			(at 67.945 204.47 0)
 			(hide yes)
 			(show_name no)
@@
 		)
 		(property "Value" "PWR_FLAG"
-			(at 67.31 204.4699 90)
+			(at 69.85 204.4699 90)
 			(show_name no)
 			(do_not_autoplace no)
@@
 		)
 		(property "Footprint" ""
-			(at 63.5 204.47 0)
+			(at 66.04 204.47 0)
 			(hide yes)
 			(show_name no)
@@
 		)
 		(property "Datasheet" ""
-			(at 63.5 204.47 0)
+			(at 66.04 204.47 0)
 			(hide yes)
 			(show_name no)
@@
 		)
 		(property "Description" "Special symbol for telling ERC where power comes from"
-			(at 63.5 204.47 0)
+			(at 66.04 204.47 0)
 			(hide yes)
 			(show_name no)
@@
 	(symbol
 		(lib_id "power:-12V")
-		(at 63.5 208.28 180)
+		(at 66.04 208.28 180)
 		(unit 1)
 		(body_style 1)
@@
 		(fields_autoplaced yes)
 		(property "Reference" "#PWR029"
-			(at 63.5 204.47 0)
+			(at 66.04 204.47 0)
 			(hide yes)
 			(show_name no)
@@
 		)
 		(property "Value" "-12V"
-			(at 63.5 213.36 0)
+			(at 66.04 213.36 0)
 			(show_name no)
 			(do_not_autoplace no)
@@
 		)
 		(property "Footprint" ""
-			(at 63.5 208.28 0)
+			(at 66.04 208.28 0)
 			(hide yes)
 			(show_name no)
@@
 		)
 		(property "Datasheet" ""
-			(at 63.5 208.28 0)
+			(at 66.04 208.28 0)
 			(hide yes)
 			(show_name no)
@@
 		)
 		(property "Description" "Power symbol creates a global label with name \"-12V\""
-			(at 63.5 208.28 0)
+			(at 66.04 208.28 0)
 			(hide yes)
 			(show_name no)
@@
 	(symbol
 		(lib_id "Device:R_US")
-		(at 234.95 137.16 90)
+		(at 234.95 137.16 270)
+		(mirror x)
 		(unit 1)
 		(body_style 1)
@@
 		(in_pos_files yes)
 		(dnp no)
-		(fields_autoplaced yes)
 		(property "Reference" "R21"
 			(at 234.95 130.81 90)
@@
 		)
 		(property "Footprint" "Resistor_THT:R_Axial_DIN0207_L6.3mm_D2.5mm_P2.54mm_Vertical"
-			(at 235.204 136.144 90)
+			(at 234.696 136.144 90)
 			(hide yes)
 			(show_name no)
@@
 	(symbol
 		(lib_id "Device:R_US")
-		(at 234.95 127 90)
+		(at 234.95 127 270)
+		(mirror x)
 		(unit 1)
 		(body_style 1)
@@
 		(in_pos_files yes)
 		(dnp no)
-		(fields_autoplaced yes)
 		(property "Reference" "R18"
 			(at 234.95 120.65 90)
@@
 		)
 		(property "Footprint" "Resistor_THT:R_Axial_DIN0207_L6.3mm_D2.5mm_P2.54mm_Vertical"
-			(at 235.204 125.984 90)
+			(at 234.696 125.984 90)
 			(hide yes)
 			(show_name no)
@@
 		(lib_id "Device:R_US")
 		(at 177.8 31.75 0)
-		(mirror x)
 		(unit 1)
 		(body_style 1)
@@
 		(dnp no)
 		(property "Reference" "R3"
-			(at 175.26 30.4799 0)
+			(at 175.26 33.0201 0)
 			(show_name no)
 			(do_not_autoplace no)
@@
 		)
 		(property "Value" "20k"
-			(at 175.26 33.0199 0)
+			(at 175.26 30.4801 0)
 			(show_name no)
 			(do_not_autoplace no)
@@
 		)
 		(property "Footprint" "Resistor_THT:R_Axial_DIN0207_L6.3mm_D2.5mm_P2.54mm_Vertical"
-			(at 178.816 31.496 90)
+			(at 178.816 32.004 90)
 			(hide yes)
 			(show_name no)
@@
 	(symbol
 		(lib_id "Device:R_US")
-		(at 69.85 35.56 90)
+		(at 69.85 35.56 270)
+		(mirror x)
 		(unit 1)
 		(body_style 1)
@@
 		(in_pos_files yes)
 		(dnp no)
-		(fields_autoplaced yes)
 		(property "Reference" "R4"
 			(at 69.85 29.21 90)
@@
 		)
 		(property "Footprint" "Resistor_THT:R_Axial_DIN0207_L6.3mm_D2.5mm_P2.54mm_Vertical"
-			(at 70.104 34.544 90)
+			(at 69.596 34.544 90)
 			(hide yes)
 			(show_name no)
@@
 	)
 	(symbol
+		(lib_id "power:PWR_FLAG")
+		(at 50.8 207.01 270)
+		(unit 1)
+		(body_style 1)
+		(exclude_from_sim no)
+		(in_bom yes)
+		(on_board yes)
+		(in_pos_files yes)
+		(dnp no)
+		(fields_autoplaced yes)
+		(property "Reference" "#FLG03"
+			(at 52.705 207.01 0)
+			(hide yes)
+			(show_name no)
+			(do_not_autoplace no)
+			(effects
+				(font
+					(size 1.27 1.27)
+				)
+			)
+		)
+		(property "Value" "PWR_FLAG"
+			(at 54.61 207.0099 90)
+			(show_name no)
+			(do_not_autoplace no)
+			(effects
+				(font
+					(size 1.27 1.27)
+				)
+				(justify left)
+			)
+		)
+		(property "Footprint" ""
+			(at 50.8 207.01 0)
+			(hide yes)
+			(show_name no)
+			(do_not_autoplace no)
+			(effects
+				(font
+					(size 1.27 1.27)
+				)
+			)
+		)
+		(property "Datasheet" ""
+			(at 50.8 207.01 0)
+			(hide yes)
+			(show_name no)
+			(do_not_autoplace no)
+			(effects
+				(font
+					(size 1.27 1.27)
+				)
+			)
+		)
+		(property "Description" "Special symbol for telling ERC where power comes from"
+			(at 50.8 207.01 0)
+			(hide yes)
+			(show_name no)
+			(do_not_autoplace no)
+			(effects
+				(font
+					(size 1.27 1.27)
+				)
+			)
+		)
+		(pin "1"
+		)
+		(instances
+			(project "DMH_Submodule_XFader"
+				(path "/58f4306d-5387-4983-bb08-41a2313fd315"
+					(reference "#FLG03")
+					(unit 1)
+				)
+			)
+		)
+	)
+	(symbol
 		(lib_id "power:GND")
 		(at 45.72 208.28 0)
@@
 	(symbol
 		(lib_id "Device:R_US")
-		(at 152.4 171.45 180)
+		(at 152.4 171.45 0)
+		(mirror y)
 		(unit 1)
 		(body_style 1)
@@
 		(in_pos_files yes)
 		(dnp no)
-		(fields_autoplaced yes)
 		(property "Reference" "R22"
-			(at 154.94 170.1799 0)
+			(at 154.94 172.7201 0)
 			(show_name no)
 			(do_not_autoplace no)
@@
 		)
 		(property "Value" "20k"
-			(at 154.94 172.7199 0)
+			(at 154.94 170.1801 0)
 			(show_name no)
 			(do_not_autoplace no)
@@
 		)
 		(property "Footprint" "Resistor_THT:R_Axial_DIN0207_L6.3mm_D2.5mm_P2.54mm_Vertical"
-			(at 151.384 171.196 90)
+			(at 151.384 171.704 90)
 			(hide yes)
 			(show_name no)
@@
 	(symbol
 		(lib_id "Device:R_US")
-		(at 152.4 31.75 180)
+		(at 152.4 31.75 0)
+		(mirror y)
 		(unit 1)
 		(body_style 1)
@@
 		(in_pos_files yes)
 		(dnp no)
-		(fields_autoplaced yes)
 		(property "Reference" "R2"
-			(at 154.94 30.4799 0)
+			(at 154.94 33.0201 0)
 			(show_name no)
 			(do_not_autoplace no)
@@
 		)
 		(property "Value" "20k"
-			(at 154.94 33.0199 0)
+			(at 154.94 30.4801 0)
 			(show_name no)
 			(do_not_autoplace no)
@@
 		)
 		(property "Footprint" "Resistor_THT:R_Axial_DIN0207_L6.3mm_D2.5mm_P2.54mm_Vertical"
-			(at 151.384 31.496 90)
+			(at 151.384 32.004 90)
 			(hide yes)
 			(show_name no)

Commit message: Xfader routing done
Parts:
- Q2: Function (none) -> 4x BC548
- RV1: Function Symmetry A -> A
- RV2: Function Symmetry B -> B
- RV3: Function Zero adj -> CV zero
Changed lines of the file:
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@@
 			)
 		)
-		(property "Function" ""
+		(property "Function" "4x BC548"
 			(at 180.34 88.9 0)
+			(hide yes)
 			(show_name no)
 			(do_not_autoplace no)
@@
 			)
 		)
-		(property "Function" "Zero adj"
+		(property "Function" "CV zero"
 			(at 88.9 27.178 90)
 			(show_name no)
@@
 			)
 		)
-		(property "Function" "Symmetry B"
-			(at 223.52 241.3 0)
+		(property "Function" "B"
+			(at 218.44 241.3 0)
 			(show_name no)
 			(do_not_autoplace no)
@@
 			)
 		)
-		(property "Function" "Symmetry A"
-			(at 223.52 101.6 0)
-			(show_name no)
-			(do_not_autoplace no)
+		(property "Function" "A"
+			(at 218.44 101.6 0)
+			(show_name no)
+			(do_not_autoplace no)

Commit message: Fixed Out A and B mix labels and routing
Connections:
- net CV Att In renamed CV_Att_In
- net CV Att Pot renamed CV_Att_Pot
- net CV Mix In renamed CV_Mix_In
- net In A renamed In_A
- net In B renamed In_B
- net Out A renamed Out_A
- net Out_A: no longer R21.2
- net Out B renamed Out_B
- net Out_B: now also R21.2
- net Out X renamed Out_X
Other:
- moved on the sheet: R18, R19, R21, R4, R5, RV3, RV4, U2A, U2B

Commit message: Swapped J1 and J2 tags around on XFader SM
Parts:
- renumbered J2 to J1, J1 to J2
Other:
- title: (none) -> Cross Fader Submodule
Changed lines of the file:
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@@
 	(paper "A3" portrait)
 	(title_block
+		(title "Cross Fader Submodule")
 		(rev "1")
 		(company "DMH Instruments")
-		(comment 1 "Cross Fader submodule for Kosmo major modules")
+		(comment 1 "Submodule PCB for Kosmo major synth modules")
 	)
 	(rectangle
@@
 		(dnp no)
 		(fields_autoplaced yes)
-		(property "Reference" "J1"
+		(property "Reference" "J2"
 			(at 66.04 170.1799 0)
 			(show_name no)
@@
 			(project "DMH_Submodule_XFader"
 				(path "/58f4306d-5387-4983-bb08-41a2313fd315"
-					(reference "J1")
+					(reference "J2")
 					(unit 1)
 				)
@@
 		(in_pos_files yes)
 		(dnp no)
-		(property "Reference" "J2"
+		(property "Reference" "J1"
 			(at 35.56 201.9299 0)
 			(show_name no)
@@
 			(project "DMH_Submodule_XFader"
 				(path "/58f4306d-5387-4983-bb08-41a2313fd315"
-					(reference "J2")
+					(reference "J1")
 					(unit 1)
 				)

Commit message: Added solder jumpers to X faders
Parts:
- added C5: 33pF, Capacitor_THT:C_Disc_D3.0mm_W2.0mm_P2.50mm, symbol Device:C
- added JP1, JP2, JP3, JP4: SolderJumper_3_Open, Jumper:SolderJumper-3_P1.3mm_Open_RoundedPad1.0x1.5mm_NumberLabels, symbol Jumper:SolderJumper_3_Open
Connections:
- net Out_X: now also C5.2
- net at Q3.1 (C), R22.2: now also JP3.3 (B), JP4.1 (A); no longer R26.2
- net at Q4.1 (C), R23.2: now also JP3.1 (A), JP4.3 (B); no longer R25.2
- net at R18.1, R19.1, R21.1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: now also C5.1
- net at Q1.1 (C), R2.2: now also JP1.3 (B), JP2.1 (A); no longer R8.2
- net at Q2.1 (C), R3.2: now also JP1.1 (A), JP2.3 (B); no longer R7.2
- new net: JP2.2 (C), R8.2
- new net: JP3.2 (C), R25.2
- new net: JP1.2 (C), R7.2
- new net: JP4.2 (C), R26.2
Other:
- note added: "Optional"
- moved on the sheet: R26, R8
